File: kicad/avr-programmer.kicad_pcb (KiCad board)
At the start: 2 copper layers, 70.4 x 54.6 mm, 12 parts, among them J1 Conn_02x14_Counter_Clockwise, J3 Conn_02x04_Counter_Clockwise, Y1 Crystal 16Mhz

Commit message: bugfix: add a capacitor to prevent programmer from resetting
Parts:
- added C1: 10uF, Capacitor_THT:C_Disc_D4.3mm_W1.9mm_P5.00mm, F.Cu at (96.5, 83.8)
- Y1: footprint Crystal:Crystal_HC49-4H_Vertical -> Crystal:Crystal_HC18-U_Vertical
- renumbered C1 to C2, C2 to C3, J3 to J2
Connections:
- A1 pad 28: unconnected-(A1-Pad28) -> Net-(A1-Pad28)
Routing:
- net Net-(A1-Pad28): track 0.00 -> 5.07 mm
